File: EverestMinishot/EverestMinishot.kicad_pcb (KiCad board)
At the start: 2 copper layers, 65 x 27 mm, 3 parts, among them J1 Conn_01x03_Pin, SW1 Mode Switch, SW2 Camera Shutter

Commit message: Updated CSV
Connections:
- net GPIO 17 renamed GPIO 4
- J1 pad 1: GND -> GPIO 3
- J1 pad 3: GPIO 27 -> GND
- SW1 pad 2: GPIO 27 -> GPIO 3
Routing:
- net GPIO 3: track 0.00 -> 26.7 mm
- net GPIO 27: track 25.9 -> 0.00 mm
Changed lines of the file:
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@@
 		(capping no)
 		(filling no)
-		(zone_defaults)
 		(pcbplotparams
 			(layerselection 0x00000000_00000000_55555555_5755f5ff)
@@
 			(layers "*.Cu" "*.Mask")
 			(remove_unused_layers no)
-			(net "GND")
+			(net "GPIO 3")
 			(pinfunction "Pin_1_1")
 			(pintype "passive")
@@
 			(layers "*.Cu" "*.Mask")
 			(remove_unused_layers no)
-			(net "GPIO 17")
+			(net "GPIO 4")
 			(pinfunction "Pin_2_2")
 			(pintype "passive")
@@
 			(layers "*.Cu" "*.Mask")
 			(remove_unused_layers no)
-			(net "GPIO 27")
+			(net "GND")
 			(pinfunction "Pin_3_3")
 			(pintype "passive")
@@
 			(layers "*.Cu" "*.Mask")
 			(remove_unused_layers no)
-			(net "GPIO 17")
+			(net "GPIO 4")
 			(pinfunction "2_2")
 			(pintype "passive")
@@
 			(layers "*.Cu" "*.Mask")
 			(remove_unused_layers no)
-			(net "GPIO 17")
+			(net "GPIO 4")
 			(pinfunction "2_2")
 			(pintype "passive")
@@
 			(layers "*.Cu" "*.Mask")
 			(remove_unused_layers no)
-			(net "GPIO 27")
+			(net "GPIO 3")
 			(pinfunction "2_2")
 			(pintype "passive")
@@
 			(layers "*.Cu" "*.Mask")
 			(remove_unused_layers no)
-			(net "GPIO 27")
+			(net "GPIO 3")
 			(pinfunction "2_2")
 			(pintype "passive")
@@
 		(end 78.5 114.5)
 		(stroke
-			(width -1)
+			(width 0.1)
 			(type default)
 		)
@@
 		(end 143.5 114.5)
 		(stroke
-			(width -1)
+			(width 0.1)
 			(type default)
 		)
@@
 		(end 79.5 90)
 		(stroke
-			(width -1)
+			(width 0.1)
 			(type default)
 		)
@@
 		(end 79.5 112)
 		(stroke
-			(width -1)
+			(width 0.1)
 			(type default)
 		)
@@
 		(end 98.087 91)
 		(stroke
-			(width -1)
+			(width 0.1)
 			(type default)
 		)
@@
 		(end 86.087 91)
 		(stroke
-			(width -1)
+			(width 0.1)
 			(type default)
 		)
@@
 		(end 98.087 103)
 		(stroke
-			(width -1)
+			(width 0.1)
 			(type default)
 		)
@@
 		(end 86.087 103)
 		(stroke
-			(width -1)
+			(width 0.1)
 			(type default)
 		)
@@
 		(end 136.187 91)
 		(stroke
-			(width -1)
+			(width 0.1)
 			(type default)
 		)
@@
 		(end 124.187 91)
 		(stroke
-			(width -1)
+			(width 0.1)
 			(type default)
 		)
@@
 		(end 136.187 103)
 		(stroke
-			(width -1)
+			(width 0.1)
 			(type default)
 		)
@@
 		(end 124.187 103)
 		(stroke
-			(width -1)
+			(width 0.1)
 			(type default)
 		)
@@
 		(end 139.5 90)
 		(stroke
-			(width -1)
+			(width 0.1)
 			(type default)
 		)
@@
 		(end 139.5 112)
 		(stroke
-			(width -1)
+			(width 0.1)
 			(type default)
 		)
@@
 		(end 78.5 87.5)
 		(stroke
-			(width -1)
+			(width 0.1)
 			(type default)
 		)
@@
 		(end 143.5 87.5)
 		(stroke
-			(width -1)
+			(width 0.1)
 			(type default)
 		)
@@
 	)
 	(segment
-		(start 105.42 101.08)
-		(end 111 101.08)
+		(start 105.5 96)
+		(end 111 96)
 		(width 0.3)
 		(layer "F.Cu")
-		(net "GPIO 27")
-	)
-	(segment
-		(start 103.5 99.5)
-		(end 105.08 101.08)
-		(width 0.3)
-		(layer "F.Cu")
-		(net "GPIO 27")
+		(net "GPIO 3")
 	)
 	(segment
 		(start 98.25 99.5)
-		(end 103.5 99.5)
+		(end 102 99.5)
 		(width 0.3)
 		(layer "F.Cu")
-		(net "GPIO 27")
+		(net "GPIO 3")
+	)
+	(segment
+		(start 102 99.5)
+		(end 105.5 96)
+		(width 0.3)
+		(layer "F.Cu")
+		(net "GPIO 3")
 	)
 	(segment
@@
 		(width 0.3)
 		(layer "F.Cu")
-		(net "GPIO 27")
+		(net "GPIO 3")
 	)
 	(segment
-		(start 105.08 101.08)
-		(end 105.42 101.08)
+		(start 111 98.54)
+		(end 115.96 98.54)
 		(width 0.3)
 		(layer "F.Cu")
-		(net "GPIO 27")
+		(net "GPIO 4")
+	)
+	(segment
+		(start 116.92 99.5)
+		(end 124 99.5)
+		(width 0.3)
+		(layer "F.Cu")
+		(net "GPIO 4")
 	)
 	(segment
 		(start 115.96 98.54)
-		(end 111 98.54)
+		(end 116.92 99.5)
 		(width 0.3)
 		(layer "F.Cu")
-		(net "GPIO 17")
-	)
-	(segment
-		(start 124 99.5)
-		(end 117 99.5)
-		(width 0.3)
-		(layer "F.Cu")
-		(net "GPIO 17")
-	)
-	(segment
-		(start 116 98.5)
-		(end 115.96 98.54)
-		(width 0.3)
-		(layer "F.Cu")
-		(net "GPIO 17")
-	)
-	(segment
-		(start 117 99.5)
-		(end 116 98.5)
-		(width 0.3)
-		(layer "F.Cu")
-		(net "GPIO 17")
+		(net "GPIO 4")
 	)
 	(segment
@@
 		(width 0.3)
 		(layer "F.Cu")
-		(net "GPIO 17")
+		(net "GPIO 4")
 	)
 	(zone
